File: FRAM01A.kicad_sch (KiCad schematic)
At the start: 8 parts

Commit message: pcb layout
Parts:
- removed J?: Conn_02x03_Odd_Even, symbol Connector_Generic:Conn_02x03_Odd_Even
- removed J?: Conn_02x05_Odd_Even, symbol Connector_Generic:Conn_02x05_Odd_Even
- added J1: HEADER_2x03_PARALLEL, Mlab_Pin_Headers:Straight_2x03, symbol MLAB_HEADER:HEADER_2x03_PARALLEL
- added J2: HEADER_2x04, Mlab_Pin_Headers:Straight_2x04, symbol MLAB_HEADER:HEADER_2x04
- H1, H2, H3, H4: renamed from H?; footprint (none) -> Mlab_Mechanical:MountingHole_3mm
- IC1: renamed from IC?; footprint SOIC127P800X203-8N -> KiCad:SOIC127P800X203-8N
- gave numbers to parts that had none: 1
Connections:
- net GND: now also J1.1, J1.2, J1.5, J1.6, J2.6, J2.8
- net MISO: now also J2.1
- net MOSI: now also J2.4
- net SCK: now also J2.3
- net VDD: now also J1.3, J1.4, J2.2
- net ~{CS}: now also J2.5
- net ~{WP}: now also J2.7
