File: hw/sch_pcb/FRAM01.kicad_sch (KiCad schematic)
At the start: 9 parts, among them IC1 CY15B108QN-40SXI, J2 HEADER_2x04, M1 HOLE M3, M2 HOLE M3, M3 HOLE, M4 HOLE

Commit message: power connection added, SPI connector changed
Parts:
- removed J2: HEADER_2x04, Mlab_Pin_Headers:Straight_2x04, symbol MLAB_HEADER:HEADER_2x04
- removed M1, M2: HOLE M3, Mlab_Mechanical:MountingHole_3mm, symbol mlab-default-rescue:HOLE
- removed M3, M4: HOLE, Mlab_Mechanical:MountingHole_3mm, symbol mlab-default-rescue:HOLE
- added J1: HEADER_2x03_PARALLEL, Mlab_Pin_Headers:Straight_2x03, symbol MLAB_HEADER:HEADER_2x03_PARALLEL
- added J2: HEADER_2x05_PARALLEL, Mlab_Pin_Headers:Straight_2x05, symbol MLAB_HEADER:HEADER_2x05_PARALLEL
- added M1, M2, M3, M4: HOLE, Mlab_Mechanical:MountingHole_3mm, symbol MLAB_MECHANICAL:HOLE
- IC1: footprint KiCad:SOIC127P800X203-8N -> SOIC127P800X203-8N; Manufacturer_Name Infineon / Cypress -> Cypress Semiconductor; Mouser Price/Stock https://www.mouser.co.uk/ProductDetail/Infineon-Cypress/CY1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 -> https://www.mouser.co.uk/ProductDetail/Cypress-Semiconducto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
Connections:
- net GND: now also J1.1, J1.2, J1.5, J1.6, M1.1, M2.1, M3.1, M4.1
- net MISO: now also J2.7, J2.8
- net MOSI: now also J2.3, J2.4
- net SCK: now also J2.1, J2.2
- net ~{CS}: now also J2.10, J2.9
- net ~{WP}: now also J2.5, J2.6
- net +3.3V renamed VDD
- net VDD: now also J1.3, J1.4
Other:
- moved on the sheet: C1, C2, D1
